File: picoEMP.kicad_sch (KiCad schematic)
At the start: 0 parts

Commit message: addede schematic components
Other:
- added sheet rp-pico2040 (rp-pico2040.kicad_sch)
- added sheet shouter (shouter.kicad_sch)
Changed lines of the file:
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@@
 	(generator_version "9.0")
 	(paper "A4")
+	(sheet
+		(at 68.58 69.85)
+		(size 43.18 31.75)
+		(exclude_from_sim no)
+		(in_bom yes)
+		(on_board yes)
+		(dnp no)
+		(fields_autoplaced yes)
+		(stroke
+			(width 0.1524)
+			(type solid)
+		)
+		(fill
+			(color 0 0 0 0.0000)
+		)
+		(property "Sheetname" "shouter"
+			(at 68.58 69.1384 0)
+			(effects
+				(font
+					(size 1.27 1.27)
+				)
+				(justify left bottom)
+			)
+		)
+		(property "Sheetfile" "shouter.kicad_sch"
+			(at 68.58 102.1846 0)
+			(effects
+				(font
+					(size 1.27 1.27)
+				)
+				(justify left top)
+			)
+		)
+		(instances
+			(project "picoEMP"
+				(path "/fd2218c3-17cf-4d7a-810a-baeaf58a762b"
+					(page "2")
+				)
+			)
+		)
+	)
+	(sheet
+		(at 121.92 71.12)
+		(size 44.45 30.48)
+		(exclude_from_sim no)
+		(in_bom yes)
+		(on_board yes)
+		(dnp no)
+		(fields_autoplaced yes)
+		(stroke
+			(width 0.1524)
+			(type solid)
+		)
+		(fill
+			(color 0 0 0 0.0000)
+		)
+		(property "Sheetname" "rp-pico2040"
+			(at 121.92 70.4084 0)
+			(effects
+				(font
+					(size 1.27 1.27)
+				)
+				(justify left bottom)
+			)
+		)
+		(property "Sheetfile" "rp-pico2040.kicad_sch"
+			(at 121.92 102.1846 0)
+			(effects
+				(font
+					(size 1.27 1.27)
+				)
+				(justify left top)
+			)
+		)
+		(instances
+			(project "picoEMP"
+				(path "/fd2218c3-17cf-4d7a-810a-baeaf58a762b"
+					(page "3")
+				)
+			)
+		)
+	)
 	(sheet_instances
 		(path "/"
