File: shouter.kicad_sch (KiCad schematic)
At the start: 27 parts, among them J1 Conn_01x02, J2 Conn_Coaxial, Q1 IPD50R3K0CE, Q2 IPD50R3K0CE, Q3 IPD50R3K0CE, SW1 SW_Push, T1 PE-68386NL, T2 PE-68386NL, U1 SFH601-2X007

Commit message: net finished, pending add shouter components any footprint
Parts:
- D1: value D_Schottky -> SM4005PL-TP
- D2: renamed from D3; value D_Schottky -> SM4005PL-TP
- D3: renamed from D2; value D_Schottky -> SM4005PL-TP
- J1: footprint (none) -> Connector_PinHeader_2.54mm:PinHeader_1x02_P2.54mm_Vertical
- Q1: renamed from Q2; value IPD50R3K0CE -> AO3422
- Q2: renamed from Q1; value IPD50R3K0CE -> AO3422
- Q3: value IPD50R3K0CE -> RGT16BM65DTL
- renumbered C2 to C1, C3 to C2, C1 to C3, R4 to R1, R5 to R2, R1 to R3, R7 to R4, R6 to R5, R9 to R6, R8 to R7, R2 to R8, R3 to R9
Connections:
- net CHARGED: now also R3.2, U1.5
- net HVPULSE: now also D3.2 (A)
- net HVPWM: now also D2.2 (A)
- net VCC: now also D1.2 (A), R3.1
- net at R4.1: now also D2.1 (K), Q1.1 (G)
- net GND: now reaches R4.2
- net GND: now also C1.2, C2.2, C3.2, Q1.3 (S), Q2.3 (S), R5.2, U1.4
- net at R1.1: now also D1.1 (K), R2.1
- net at R1.2: now also C1.1, C3.1, T1.3
- net at R5.1: now also D3.1 (K), Q2.1 (G)
- net at T2.1: now also Q2.2 (D)
- net at T2.3: now also C2.1, R2.2
- net at Q1.2 (D): now also T1.1
Other:
- moved on the sheet: C1, C2, C3, D3, Q1, R3, R5

Commit message: update components, pending route signals of connectors
Parts:
- renumbered C3 to C1, C1 to C2, C2 to C3, D3 to D2, D2 to D3, Q2 to Q1, Q1 to Q2, R3 to R1, R8 to R2, R9 to R3, R1 to R4, R2 to R5, R5 to R6, R4 to R7, R7 to R8, R6 to R9
Changed lines of the file:
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@@
 		(dnp no)
 		(fields_autoplaced yes)
-		(property "Reference" "R4"
+		(property "Reference" "R7"
 			(at 87.63 99.0599 0)
 			(effects
@@
 		(dnp no)
 		(fields_autoplaced yes)
-		(property "Reference" "D2"
+		(property "Reference" "D3"
 			(at 77.7875 86.36 0)
 			(effects
@@
 		(dnp no)
 		(fields_autoplaced yes)
-		(property "Reference" "R9"
+		(property "Reference" "R3"
 			(at 186.69 58.4199 0)
 			(effects
@@
 		(dnp no)
 		(fields_autoplaced yes)
-		(property "Reference" "R7"
+		(property "Reference" "R8"
 			(at 158.75 119.38 90)
 			(effects
@@
 		(dnp no)
 		(fields_autoplaced yes)
-		(property "Reference" "R1"
+		(property "Reference" "R4"
 			(at 63.5 72.39 90)
 			(effects
@@
 		(dnp no)
 		(fields_autoplaced yes)
-		(property "Reference" "#PWR03"
+		(property "Reference" "#PWR?"
 			(at 107.95 170.18 0)
 			(effects
@@
 				(path "/86f9a32b-85fd-41b7-9dca-384e1cbe91ec"
 					(reference "#PWR03")
+					(unit 1)
+				)
+			)
+			(project "picoEMP"
+				(path "/fd2218c3-17cf-4d7a-810a-baeaf58a762b/09f6e0cf-af80-4f7b-8458-c3eb185fcadf"
+					(reference "#PWR?")
 					(unit 1)
 				)
@@
 		(dnp no)
 		(fields_autoplaced yes)
-		(property "Reference" "#PWR05"
+		(property "Reference" "#PWR01"
 			(at 77.47 39.37 0)
 			(effects
@@
 		(dnp no)
 		(fields_autoplaced yes)
-		(property "Reference" "R5"
+		(property "Reference" "R6"
 			(at 90.17 149.8599 0)
 			(effects
@@
 		(dnp no)
 		(fields_autoplaced yes)
-		(property "Reference" "R8"
+		(property "Reference" "R2"
 			(at 173.99 44.45 90)
 			(effects
@@
 		(on_board yes)
 		(dnp no)
-		(property "Reference" "C1"
+		(property "Reference" "C2"
 			(at 111.76 100.3299 0)
 			(effects
@@
 		(dnp no)
 		(fields_autoplaced yes)
-		(property "Reference" "#PWR01"
+		(property "Reference" "#PWR?"
 			(at 120.65 67.31 0)
 			(effects
@@
 				)
 			)
+			(project "picoEMP"
+				(path "/fd2218c3-17cf-4d7a-810a-baeaf58a762b/09f6e0cf-af80-4f7b-8458-c3eb185fcadf"
+					(reference "#PWR?")
+					(unit 1)
+				)
+			)
 		)
 	)
@@
 		(on_board yes)
 		(dnp no)
-		(property "Reference" "C3"
+		(property "Reference" "C1"
 			(at 128.778 100.076 0)
 			(effects
@@
 		(dnp no)
 		(fields_autoplaced yes)
-		(property "Reference" "#PWR02"
+		(property "Reference" "#PWR?"
 			(at 105.41 119.38 0)
 			(effects
@@
 				)
 			)
+			(project "picoEMP"
+				(path "/fd2218c3-17cf-4d7a-810a-baeaf58a762b/09f6e0cf-af80-4f7b-8458-c3eb185fcadf"
+					(reference "#PWR?")
+					(unit 1)
+				)
+			)
 		)
 	)
@@
 		(dnp no)
 		(fields_autoplaced yes)
-		(property "Reference" "#PWR04"
+		(property "Reference" "#PWR02"
 			(at 39.37 90.17 0)
 			(effects
@@
 		(on_board yes)
 		(dnp no)
-		(property "Reference" "Q2"
+		(property "Reference" "Q1"
 			(at 111.76 142.2399 0)
 			(effects
@@
 		(dnp no)
 		(fields_autoplaced yes)
-		(property "Reference" "R3"
+		(property "Reference" "R1"
 			(at 80.01 41.9099 0)
 			(effects
@@
 		(dnp no)
 		(fields_autoplaced yes)
-		(property "Reference" "D3"
+		(property "Reference" "D2"
 			(at 79.0575 137.16 0)
 			(effects
@@
 		(dnp no)
 		(fields_autoplaced yes)
-		(property "Reference" "R6"
+		(property "Reference" "R9"
 			(at 151.13 130.8099 0)
 			(effects
@@
 		(on_board yes)
 		(dnp no)
-		(property "Reference" "Q1"
+		(property "Reference" "Q2"
 			(at 109.22 91.4399 0)
 			(effects
@@
 		(dnp no)
 		(fields_autoplaced yes)
-		(property "Reference" "C2"
+		(property "Reference" "C3"
 			(at 124.46 149.8599 0)
 			(effects
@@
 		(dnp no)
 		(fields_autoplaced yes)
-		(property "Reference" "R2"
+		(property "Reference" "R5"
 			(at 64.77 118.11 90)
 			(effects

Commit message: update components and footprints
Parts:
- C1, C2: PART_NUMBER_LCSC (none) -> C51205
- C3: PART_NUMBER_LCSC (none) -> C24497
- C4: PART_NUMBER_LCSC (none) -> C106147
- D1, D2, D3: footprint (none) -> Diode_SMD:Nexperia_CFP3_SOD-123W; PART_NUMBER_LCSC (none) -> C330237
- D4: PART_NUMBER_LCSC (none) -> C50432
- D5: footprint Diode_THT:D_DO-41_SOD81_P10.16mm_Horizontal -> Diode_SMD:Nexperia_CFP3_SOD-123W; PART_NUMBER_LCSC (none) -> C891584
- J2: footprint (none) -> Connector_Coaxial:SMA_Amphenol_132289_EdgeMount
- Q1, Q2: footprint Package_TO_SOT_SMD:TO-252-2 -> Package_TO_SOT_SMD:SOT-23; PART_NUMBER_LCSC (none) -> C37130
- Q3: PART_NUMBER_LCSC (none) -> C3193927
- R1: PART_NUMBER_LCSC (none) -> C1409
- R2: PART_NUMBER_LCSC (none) -> C71198
- R3, R4: PART_NUMBER_LCSC (none) -> C17954
- R5, R8: PART_NUMBER_LCSC (none) -> C17903
- R6, R7: PART_NUMBER_LCSC (none) -> C4410
- R9: PART_NUMBER_LCSC (none) -> C17944
- SW1: footprint (none) -> Button_Switch_SMD:SW_SPST_CK_RS282G05A3; PART_NUMBER_LCSC (none) -> C318938
- T1, T2: PART_NUMBER_LCSC (none) -> C581397
- U1: PART_NUMBER_LCSC (none) -> C17237090

Commit message: 'pads_añadidos'
Connections:
- net at U1.1: now also R2.2; no longer R2.1
- net at J1.2 (Pin_2), R3.1, SW1.2: now also R2.1; no longer R2.2
Other:
- moved on the sheet: R2
Changed lines of the file:
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@@
 	(symbol
 		(lib_id "Device:R")
-		(at 173.99 50.8 90)
+		(at 173.99 50.8 270)
+		(mirror x)
 		(unit 1)
 		(exclude_from_sim no)
@@
 		(on_board yes)
 		(dnp no)
-		(fields_autoplaced yes)
 		(property "Reference" "R2"
 			(at 173.99 44.45 90)
